File: board_design/Spring12_6/Spring12_6_Node.sch (EAGLE design)
At the start: 29 parts, among them Q1 20MHz, X1 1751248

Commit message: PCB Rev 0 done
Parts:
- removed LED1, LED2, LED3, LED4, LED5, LED6: (no value), led:LED3MM
- removed SV3: GPSR, con-lstb:MA06-1
- removed U$18, U$19, U$20, U$21: 100, 4534_I2C2:R-1/4W
- added 76SC03T: I2C Select, ic-package:DIL6
- added DB0, DB1, DB2, DB3, GPS-LED, PWR-LED: LED-SMD-1206, 4534_I2C2:LED-SMD-1206
- added IC1: L78S05CV, v-reg:78XXL
- added JP2: GPSR, pinhead:PINHD-1X6/90
- added SV6: I2C BUS, 4534_I2C2:MA07-1
- added U$2, U$3: 1k, 4534_I2C2:R-1/4W
- added U$22, U$23: 1N5817P, 4534_I2C2:1N5817P
- added U$25: EVQ-11U05R, 4534_Node_Board:EVQ-11U05R
- added U$26: 0.33uF, 4534_I2C2:C2.5-5
- added U$27: 0.1uF, 4534_I2C2:C2.5-5
- added U$28: 7-361-BA, 4534_Node_Board:7-361-BA
- added U$4, U$5: 330, 4534_I2C2:R-1/4W
- added U$6, U$7: 100pF, 4534_I2C2:C2.5-5
- SV2: value POWER SEL -> PWR CNTL; device con-lstb:MA03-1 -> con-lstb:MA03-2
- U$17: value 100 -> 2479-BATTERY; device 4534_I2C2:R-1/4W -> 4534_Node_Board:2479-BATTERY
Connections:
- removed net 3V: JP1.2, SV3.4, SV4.10, SV5.9, U$1.VDD, U$1.VDD_2, U$10.P$1, U$11.VIN, U$14.SENSE, U$14.VOUT, U$16.1
- removed net 3V-BACKUP: SV3.5
- removed net MRF-CS: U$11.~CS
- removed net N$10: LED5.C, LED6.C
- removed net N$11: SV5.20, U$1.RD2/PSP2/SDO2
- removed net N$19: SV4.13
- removed net N$24: SV4.6
- removed net N$25: SV4.5
- removed net N$4: LED2.A, U$18.2
- removed net N$5: LED6.A, U$21.2
- removed net N$9: SV5.19, U$1.RD3/PSP3/*SS2
- removed net V-EXT: X1-2.K
- new net 3V3: 76SC03T.4, 76SC03T.6, JP2.3, SV4.10, SV5.9, U$1.VDD, U$1.VDD_2, U$10.P$1, U$11.VIN, U$14.SENSE, U$14.VOUT, U$16.1, U$2.2, U$3.2
- new net 3V3-REG: SV2.4, U$14.*SHDN, U$14.VIN, U$14.VIN_2, U$15.1
- net 5V: now also IC1.OUT, JP1.2, SV2.6, SV6.3, SV6.4, SV6.5, U$27.1, U$4.2, U$5.2, U$9.VCC
- net BATTERY: now also JP2.2, U$17.VCC
- net CURRENT: now also SV2.3; no longer SV2.2
- net DB-LED0: now also DB0.A; no longer U$17.1
- net DB-LED1: now also DB1.A; no longer U$18.1
- net DB-LED2: now also DB2.A; no longer U$19.1
- net DB-LED3: now also DB3.A; no longer U$20.1
- net EXTERNAL: now also SV2.5, X1-2.K; no longer SV2.3
- net GPS-LED: now also GPS-LED.A, JP2.1; no longer LED5.A, SV3.6
- net I2C-ADDR0: now also 76SC03T.2
- net I2C-ADDR1: now also 76SC03T.5
- net MRF-RESET: now also SV5.19, U$1.RD3/PSP3/*SS2
- net MRF-WAKE: now also SV5.20, U$1.RD2/PSP2/SDO2
- net N$1: now also SV4.13, U$1.RE0/*RD/AN5; no longer LED1.A, U$17.2
- net N$2: now also SV4.6, U$1.RC0/T1OSO/T1CKI; no longer LED3.A, U$19.2
- net N$3: now also SV4.5, U$1.RC1/T1OSI/CCP2; no longer LED4.A, U$20.2
- net PIC-RESET: now also U$25.MOMENTARY
- net PWR-LED: now also PWR-LED.A; no longer U$21.1
- net REGULATORS: now also IC1.IN, SV2.2, U$26.1; no longer U$14.*SHDN, U$14.VIN, U$14.VIN_2, U$15.1
- net SCL-BUS: now also SV6.2, U$22.C, U$4.1
- net SCL-LOCAL: now also U$2.1, U$7.2
- net SDA-BUS: now also SV6.6, U$23.C, U$5.1
- net SDA-LOCAL: now also U$3.1, U$6.2
- net UART-RX: now also JP2.5; no longer SV3.2
- net UART-TX: now also JP2.6; no longer SV3.1
- net VSS: now also 76SC03T.1, 76SC03T.3, DB0.C, DB1.C, DB2.C, DB3.C, GPS-LED.C, IC1.GND, JP2.4, PWR-LED.C, SV6.1, SV6.7, U$11.~CS, U$17.VSS, U$22.A, U$23.A, U$25.SIGNAL, U$26.2, U$27.2, U$6.1, U$7.1, U$9.GND; no longer LED1.C, LED2.C, LED3.C, LED4.C, SV3.3
Other:
- note added: "20MHz Crystal Oscillator"
- note added: "5V Regulator 2A Max"
- note added: "Current Test Port"
- note added: "Dual Headers to support NODE0"
- note added: "External Power Connector"
- note added: "MCP1725-3302E/SN"
- note added: "MRF24J40MA MiWi Module"
- note added: "Power Select Jumpers"
- note removed: "Green PWR LED"
- note removed: "MCP1725-3002E/SN"
- note removed: "Orange GPS Fix LED"
- note removed: "Red Debug LEDs"
- moved on the sheet: SV1, SV5, U$8

Commit message: PCB V2
Connections:
- net N$26: now also U$1.RC2/CCP1/P1A
Other:
- note added: "On Battery: 1-3 2-4 Jumpered"
- note added: "On External: 5-3 6-4 Jumpered"
- note added: "On I2C: 5-3 6-4 Jumpered"
Changed lines of the file:
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@@
 <text x="-172.72" y="38.1" size="1.778" layer="91">Dual Headers to support NODE0</text>
 <text x="53.34" y="93.98" size="1.778" layer="91">5V Regulator 2A Max</text>
+<text x="-27.94" y="17.78" size="1.778" layer="91">On Battery: 1-3 2-4 Jumpered</text>
+<text x="-27.94" y="15.24" size="1.778" layer="91">On External: 5-3 6-4 Jumpered</text>
+<text x="-27.94" y="12.7" size="1.778" layer="91">On I2C: 5-3 6-4 Jumpered</text>
 </plain>
 <instances>
@@
 <pinref part="SV4" gate="1" pin="4"/>
 <wire x1="-147.32" y1="88.9" x2="-127" y2="88.9" width="0.1524" layer="91"/>
-</segment>
-</net>
+<pinref part="U$1" gate="A" pin="RC2/CCP1/P1A"/>
+</segment>
+</net>

Commit message: pcb stuff >_>
Parts:
- removed JP1: PICKIT, pinhead:PINHD-1X6/90
- removed JP2: GPSR, pinhead:PINHD-1X6/90
- removed SV4, SV5: (no value), con-lstb:MA20-1
- removed U$1: PIC18F45J10-X/P, 4534_Node_Board:PIC18F45J10-X/P
- removed U$25: EVQ-11U05R, 4534_Node_Board:EVQ-11U05R
- added C10: 10uF, 4534_I2C2:C2.5-5
- added C11, C8, C9: 0.1uF, 4534_I2C2:C2.5-5
- added J0, J1: (no value), con-lstb:MA20-1
- added J3: PICKIT, 4534:MA06-1
- added J6: GPSR, 4534:MA06-1
- added PIC0: PIC18F45J10-I/P, 4534:PIC18F45J10-I/P
- added R10, R11, R8, R9: 150, 4534_I2C2:R1206
- added R4: 10k, 4534_I2C2:R1206
- added R5: 100, 4534_I2C2:R1206
- added R6, R7: 60, 4534_I2C2:R1206
- added SW0: SW-PB-MOM, 4534:SW-PB-MOM
- added U$18, U$19, U$20: VIA, 4534_I2C2:VIA
- C2, C3: value 18pF -> 9pF
- C4, C5: value 100pF -> 220pF
- SW1: value I2C Select -> 76SC03T
- renumbered 76SC03T to SW1, IC1 to REG1, SV1 to J4, SV2 to J8, SV6 to J5, U$10 to J2, U$11 to RF0, U$12 to C3, U$13 to C2, U$14 to REG0, U$15 to C6, U$16 to C7, U$17 to BATT0, U$2 to R1, U$22 to D1, U$23 to D0, U$26 to C0, U$27 to C1, U$3 to R0, U$4 to R2, U$5 to R3, U$6 to C4, U$7 to C5, U$8 to J9, U$9 to IC0, X1 to J7
Connections:
- new net N$10: DB2.A, R10.2
- new net N$11: DB3.A, R11.2
- new net N$4: GPS-LED.A, R6.2
- new net N$5: PWR-LED.A, R7.2
- new net N$6: C11.1, R4.1, R5.1, SW0.S
- new net N$7: DB0.A, R8.2
- new net N$9: DB1.A, R9.2
- net 3V3: now also C8.1, C9.1, J0.11, J1.12, J6.4, PIC0.VDD, PIC0.VDD@1, R4.2; no longer JP2.3, SV4.10, SV5.9, U$1.VDD, U$1.VDD_2
- net 5V: now also J3.2; no longer JP1.2
- net BATTERY: now also J6.5; no longer JP2.2
- net DB-LED0: now also J1.14, PIC0.RB1/INT1/AN10, R8.1; no longer DB0.A, SV5.7, U$1.RB1/INT1/AN10
- net DB-LED1: now also J1.15, PIC0.RB2/INT2/AN8, R9.1; no longer DB1.A, SV5.6, U$1.RB2/INT2/AN8
- net DB-LED2: now also J1.16, PIC0.RB3/AN9/CCP2, R10.1; no longer DB2.A, SV5.5, U$1.RB3/AN9/CCP2
- net DB-LED3: now also J1.17, PIC0.RB4/KBI0/AN11, R11.1; no longer DB3.A, SV5.4, U$1.RB4/KBI0/AN11
- net GPS-LED: now also J6.6, R6.1; no longer GPS-LED.A, JP2.1
- net I2C-ADDR0: now also J1.8, PIC0.RD5/PSP5/P1B; no longer SV5.13, U$1.RD5/PSP5/P1B
- net I2C-ADDR1: now also J1.9, PIC0.RD6/PSP6/P1C; no longer SV5.12, U$1.RD6/PSP6/P1C
- net I2C-ADDR2: now also J1.10, PIC0.RD7/PSP7/P1D; no longer SV5.11, U$1.RD7/PSP7/P1D
- net MRF-INT: now also J1.13, PIC0.RB0/INT0/FLT0/AN12; no longer SV5.8, U$1.RB0/INT0/FLT0/AN12
- net MRF-RESET: now also J1.2, PIC0.RD3/PSP3/!SS2!; no longer SV5.19, U$1.RD3/PSP3/*SS2
- net MRF-WAKE: now also J1.1, PIC0.RD2/PSP2/SDO2; no longer SV5.20, U$1.RD2/PSP2/SDO2
- net N$1: now also J0.8, PIC0.RE0/!RD!/AN5; no longer SV4.13, U$1.RE0/*RD/AN5
- net N$13: now also J0.2, PIC0.RA0/AN0; no longer SV4.19, U$1.RA0/AN0
- net N$14: now also J0.3, PIC0.RA1/AN1; no longer SV4.18, U$1.RA1/AN1
- net N$15: now also J0.4, PIC0.RA2/AN2/VREF-/CVREF; no longer SV4.17, U$1.RA2/AN2/VREF-/CVREF
- net N$16: now also J0.5, PIC0.RA3/AN3/VREF+; no longer SV4.16, U$1.RA3/AN3/VREF+
- net N$17: now also C10.1, J0.6, PIC0.VDDCORE/VCAP; no longer SV4.15, U$1.VDDCORE/VCAP
- net N$18: now also J0.7, PIC0.RA5/AN4/!SS1!/C2OUT; no longer SV4.14, U$1.RA5/AN4/*SS1/C2OUT
- net N$2: now also J0.15, PIC0.RC0/T1OSO/T1CKI; no longer SV4.6, U$1.RC0/T1OSO/T1CKI
- net N$20: now also J0.9, PIC0.RE1/!WR!/AN6; no longer SV4.12, U$1.RE1/*WR/AN6
- net N$21: now also J0.10, PIC0.RE2/!CS!/AN7; no longer SV4.11, U$1.RE2/*CS/AN7
- net N$26: now also J0.17, PIC0.RC2/CCP1/P1A; no longer SV4.4, U$1.RC2/CCP1/P1A
- net N$3: now also J0.16, PIC0.RC1/T1OSI/CCP2; no longer SV4.5, U$1.RC1/T1OSI/CCP2
- net N$8: now also J1.7, PIC0.RD4/PSP4; no longer SV5.14, U$1.RD4/PSP4
- net OSC1: now also J0.13, PIC0.OSC1/CLKI; no longer SV4.8, U$1.OSC1/CLKI
- net OSC2: now also J0.14, PIC0.OSC2/CLKO; no longer SV4.7, U$1.OSC2/CLKO
- net PGC: now also J1.19, J3.5, PIC0.RB6/KBI2/PGC; no longer JP1.5, SV5.2, U$1.RB6/KBI2/PGC
- net PGD: now also J1.20, J3.4, PIC0.RB7/KBI3/PGD; no longer JP1.4, SV5.1, U$1.RB7/KBI3/PGD
- net PIC-RESET: now also J0.1, J3.1, PIC0.!MCLR!/VPP/RE3, R5.2; no longer JP1.1, SV4.20, U$1.*MCLR, U$25.MOMENTARY
- net PICKIT-AUX: now also J3.6; no longer JP1.6
- net PWR-LED: now also J1.18, PIC0.RB5/KBI1/TOCKI/C1OUT, R7.1; no longer PWR-LED.A, SV5.3, U$1.RB5/KBI1/T0CKI/C1OUT
- net SCL-LOCAL: now also J0.19, PIC0.RD0/PSP0/SCK2/SCL2; no longer SV4.2
- net SDA-LOCAL: now also J0.20, PIC0.RD1/PSP1/SDI2/SDA2; no longer SV4.1, U$1.RD1/PSP1/SDI2/SDA2
- net SPI-MISO: now also J1.3, PIC0.RC4/SDI1/SDA1; no longer SV5.18, U$1.RC4/SDI1/SDA1
- net SPI-MOSI: now also J1.4, PIC0.RC5/SDO1; no longer SV5.17, U$1.RC5/SDO1
- net SPI-SCK: now also J0.18, PIC0.RC3/SCK1/SCL1; no longer SV4.3, U$1.RC3/SCK1/SCL1
- net UART-RX: now also J1.6, J6.2, PIC0.RC7/RX/DT; no longer JP2.5, SV5.15, U$1.RC7/RX/DT
- net UART-TX: now also J1.5, J6.1, PIC0.RC6/TX/CK; no longer JP2.6, SV5.16, U$1.RC6/TX/CK
- net VSS: now also C10.2, C11.2, C8.2, C9.2, J0.12, J1.11, J3.3, J6.3, PIC0.VSS, PIC0.VSS@1, SW0.P, U$18.P, U$19.P, U$20.P; no longer JP1.3, JP2.4, SV4.9, SV5.10, U$1.VSS, U$1.VSS_2, U$25.SIGNAL
Other:
- note added: "I2C Select"
- moved on the sheet: DB0, DB1, DB2, DB3
