File: board_design/Spring12_6_daughterboard/Spring12_6_daughterboard.brd (EAGLE design)
At the start: 28.9 x 52.1 mm, 4 parts

Commit message: changed project requirements document
Parts:
- added R1: 560, rcl:R1206
- moved PPS-LED 3.81 mm to (27.9, 8.89)
Connections:
- new net N$1: PPS-LED.A, R1.2
- net GPS-LED: now also R1.1; no longer PPS-LED.A
Routing:
- net N$1: track 0.00 -> 7.62 mm
- net GPS-LED: track 10.6 -> 15.2 mm
- net VSS: track 6.83 -> 10.6 mm
Other:
- board size 28.9 x 52.1 mm -> 34 x 52.1 mm
Changed lines of the file:
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@@
 <layer number="43" name="vRestrict" color="2" fill="10" visible="yes" active="yes"/>
 <layer number="44" name="Drills" color="7" fill="1" visible="no" active="yes"/>
-<layer number="45" name="Holes" color="7" fill="1" visible="no" active="yes"/>
+<layer number="45" name="Holes" color="7" fill="1" visible="yes" active="yes"/>
 <layer number="46" name="Milling" color="3" fill="1" visible="no" active="yes"/>
 <layer number="47" name="Measures" color="7" fill="1" visible="no" active="yes"/>
@@
 <board>
 <plain>
-<wire x1="0" y1="0" x2="28.88" y2="0" width="0" layer="20"/>
-<wire x1="28.88" y1="0" x2="28.88" y2="52.06" width="0" layer="20"/>
-<wire x1="28.88" y1="52.06" x2="0" y2="52.06" width="0" layer="20"/>
+<wire x1="0" y1="0" x2="33.96" y2="0" width="0" layer="20"/>
+<wire x1="33.96" y1="0" x2="33.96" y2="52.06" width="0" layer="20"/>
+<wire x1="33.96" y1="52.06" x2="0" y2="52.06" width="0" layer="20"/>
 <wire x1="0" y1="52.06" x2="0" y2="0" width="0" layer="20"/>
-<text x="15.24" y="44.45" size="0.8128" layer="21">ECE4534 - Group 6</text>
-<text x="15.24" y="43.18" size="0.8128" layer="21">Spring 2012</text>
-<text x="15.24" y="41.91" size="0.8128" layer="21">MiWi Daughterboard</text>
+<text x="6.35" y="44.45" size="0.8128" layer="21">ECE4534 - Group 6</text>
+<text x="6.35" y="43.18" size="0.8128" layer="21">Spring 2012</text>
+<text x="6.35" y="41.91" size="0.8128" layer="21">MiWi Daughterboard</text>
+<hole x="26.67" y="41.91" drill="6.3754"/>
+<rectangle x1="3.81" y1="15.24" x2="25.4" y2="35.56" layer="41"/>
 </plain>
 <attributes>
@@
 <attribute name="NAME" x="8.89" y="12.7" size="1.016" layer="26" font="vector" ratio="15" rot="MR180"/>
 </element>
-<element name="PPS-LED" library="4534_I2C2" package="LED1206" value="LED-SMD-1206" x="24.13" y="8.89" smashed="yes" rot="R180">
-<attribute name="NAME" x="26.67" y="3.81" size="1.27" layer="25" font="vector" ratio="15" rot="R90"/>
+<element name="PPS-LED" library="4534_I2C2" package="LED1206" value="LED-SMD-1206" x="27.94" y="8.89" smashed="yes" rot="R180">
+<attribute name="NAME" x="30.48" y="3.81" size="1.27" layer="25" font="vector" ratio="15" rot="R90"/>
 </element>
 <element name="U$1" library="4534_Node_Board" package="796136-1-CR2032_HOLDER" value="796136-1-CR2302_HOLDER" x="13.97" y="27.94" rot="MR90"/>
 <element name="U$3" library="4534_Node_Board" package="GPS-UP501" value="GPS-UP501" x="12.7" y="20.32"/>
+<element name="R1" library="rcl" package="R1206" value="560" x="27.94" y="19.05" rot="R270"/>
 </elements>
 <signals>
@@
 <polygon width="0.4064" layer="16">
 <vertex x="0" y="52.07"/>
-<vertex x="29.21" y="52.07"/>
-<vertex x="29.21" y="0"/>
+<vertex x="34.29" y="52.07"/>
+<vertex x="34.29" y="0"/>
 <vertex x="0" y="0"/>
 </polygon>
-<wire x1="17.78" y1="7.62" x2="24.13" y2="7.62" width="0.254" layer="1"/>
-<wire x1="24.13" y1="7.62" x2="24.13" y2="7.14" width="0.254" layer="1"/>
+<wire x1="17.78" y1="7.62" x2="27.94" y2="7.62" width="0.254" layer="1"/>
+<wire x1="27.94" y1="7.62" x2="27.94" y2="7.14" width="0.254" layer="1"/>
 </signal>
 <signal name="BATTERY">
@@
 <signal name="GPS-LED">
 <contactref element="U$3" pad="P$6"/>
-<contactref element="PPS-LED" pad="A"/>
-<wire x1="17.78" y1="10.16" x2="24.13" y2="10.16" width="0.254" layer="1"/>
-<wire x1="17.78" y1="13.97" x2="17.78" y2="10.16" width="0.254" layer="1"/>
-<wire x1="24.13" y1="10.16" x2="24.13" y2="10.64" width="0.254" layer="1"/>
+<contactref element="R1" pad="1"/>
+<wire x1="26.67" y1="19.05" x2="27.94" y2="20.32" width="0.254" layer="1"/>
+<wire x1="26.67" y1="15.24" x2="26.67" y2="19.05" width="0.254" layer="1"/>
+<wire x1="25.4" y1="13.97" x2="26.67" y2="15.24" width="0.254" layer="1"/>
+<wire x1="17.78" y1="13.97" x2="25.4" y2="13.97" width="0.254" layer="1"/>
+<wire x1="27.94" y1="20.32" x2="27.94" y2="20.472" width="0.254" layer="1"/>
 </signal>
 <signal name="SPI_MISO">
@@
 <contactref element="U$3" pad="P$4"/>
 <wire x1="16.51" y1="6.35" x2="17.78" y2="5.08" width="0.254" layer="1"/>
-<wire x1="16.51" y1="8.89" x2="16.51" y2="6.35" width="0.254" layer="1"/>
-<wire x1="12.7" y1="12.7" x2="16.51" y2="8.89" width="0.254" layer="1"/>
-<wire x1="12.7" y1="13.97" x2="12.7" y2="12.7" width="0.254" layer="1"/>
+<wire x1="16.51" y1="10.16" x2="16.51" y2="6.35" width="0.254" layer="1"/>
+<wire x1="12.7" y1="13.97" x2="16.51" y2="10.16" width="0.254" layer="1"/>
 </signal>
 <signal name="GPIO">
 <contactref element="ACCESSORY" pad="8"/>
 </signal>
+<signal name="N$1">
+<contactref element="PPS-LED" pad="A"/>
+<contactref element="R1" pad="2"/>
+<wire x1="27.94" y1="17.628" x2="27.94" y2="10.64" width="0.254" layer="1"/>
+<wire x1="27.94" y1="10.16" x2="27.94" y2="10.64" width="0.254" layer="1"/>
+<wire x1="27.94" y1="17.78" x2="27.94" y2="17.628" width="0.254" layer="1"/>
+</signal>
 </signals>
