File: board_design/Spring12_6_rev4/Spring12_6_rev4.brd (EAGLE design)
At the start: 100 x 80.6 mm, 48 parts, among them IC1 LM555D, J3 PICKIT, Q1 20MHz, SW0 SW-PB-MOM

Commit message: board design... hopefully done
Parts:
- added C15: 100pF, rcl:C1206
- added F1: 1A PTC, SparkFun:PTC-1206
- added J1, J2: (no value), 4534:MA07-1
- added L1: 10nH, rcl:L1812
- added POWER: MA02-1, 4534:MA02-1
- added SV3, SV4, SV5: (no value), 4534:MA03-1
- added U$3, U$4, U$5: VIA, 4534_I2C2:VIA
- R5, R6: value 4K7 -> 10K
- U$2: value NHD-C0216CIZ-FN-FBW-3V -> NHD-C0216CIZ-FSW-FBW-3V3
- moved BACKLIGHT 53.4 mm to (69.2, 77.5), turned to 90 degrees
- moved C13 30.7 mm to (99.1, 44.5), turned to 270 degrees
- moved U$2 27.5 mm to (97.2, 44.5), turned to 90 degrees
- moved C12 27.4 mm to (99.1, 48.9), turned to 90 degrees
- moved J3 20.4 mm to (52.1, 80.6), flipped to the top, turned to 0 degrees
- moved R5 10.2 mm to (66.0, 60.3), turned to 270 degrees
- moved ACCESSORY-1 8.82 mm to (94.0, 11.4), turned to 270 degrees
- moved ACCESSORY-2 7.41 mm to (82.5, 11.4), turned to 270 degrees
- moved C1 7.24 mm to (40.6, 37.5), turned to 90 degrees
- moved C5 4.26 mm to (48.3, 24.1), turned to 270 degrees
- moved R6 4.07 mm to (62.2, 60.3)
- moved U$18 2.84 mm to (3.81, 10.8)
- moved U$19 1.42 mm to (3.81, 32.4)
- moved C2 0.64 mm to (27.9, 37.5)
- moved U$20 0.64 mm to (13.3, 33.0)
Connections:
- removed net 5V: J3.2
- new net BATT: BATT0.P$2, F1.2
- new net CURRENT: J2.3, J2.4, J2.5, SV3.1, SV4.1, SV5.1
- new net MIWI-VDD: C15.1, L1.1, RF0.10
- new net N$12: F1.1, POWER.1
- new net N$14: J1.2
- new net N$17: J2.6
- new net N$21: J2.2
- new net N$7: J1.6
- new net VCC_REG0: C5.1, REG0.1, REG0.2, REG0.3, SV3.2
- new net VCC_REG1: C1.1, REG1.1, REG1.2, REG1.3, SV4.2
- new net VCC_REG2: C3.1, REG2.1, REG2.2, REG2.3, SV5.2
- net VCC_BATT: now also J1.3, J1.4, J1.5, POWER.2, SV3.3, SV4.3, SV5.3; no longer BATT0.P$2, C1.1, C3.1, C5.1, REG0.1, REG0.2, REG0.3, REG1.1, REG1.2, REG1.3, REG2.1, REG2.2, REG2.3
- net VDD_ACC: now also U$2.5, U$3.1, U$4.1
- net VDD_MIWI: now also L1.2, U$5.1; no longer RF0.10
- net VDD_PIC: now also J3.2; no longer U$2.5
- net VSS: now also C15.2, J1.1, J1.7, J2.1, J2.7
Routing:
- net SPI_MOSI: track 220.5 -> 144.3 mm, vias 3 -> 2
- net UART_TX: track 156.3 -> 197.3 mm, vias 3 -> 5
- net VDD_PIC: track 171.1 -> 135.2 mm, vias 3 -> 5
- net PGD: track 67.5 -> 31.6 mm
- net VCC_BATT: track 69.9 -> 34.3 mm
- net VCC_REG2: track 0.00 -> 32.9 mm
- net SPI_SCK: track 191.3 -> 158.5 mm, vias 1 -> 4
- net CURRENT: track 0.00 -> 24.5 mm
- net VDD_ACC: track 133.7 -> 110.4 mm, vias 2 -> 1
- net UART_RX: track 113.6 -> 136.8 mm, vias 4 -> 2
- net MCLR: track 38.4 -> 15.3 mm
- net SPI_MISO: track 130.5 -> 111.6 mm, vias 3 -> 4
- net I2C_SCL: track 148.1 -> 165.8 mm, vias 5 -> 4
- net MRF-WAKE: track 69.9 -> 85.7 mm, vias 2 -> 1
- net I2C_SDA: track 148.4 -> 132.7 mm, vias 4 -> 3
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Other:
- board size 100 x 80.6 mm -> 101.3 x 82.5 mm
- board text added: "CURRENT-0"
- board text added: "CURRENT-1"
- board text added: "CURRENT-2"
- board text added: "MCP1725"
- board text added: "Measure Current"
- board text added: "Normal"

Commit message: more PCB revs
Parts:
- F1: value 1A PTC -> 2.2A PTC
Connections:
- new net PICKIT-VDD: J3.2
- net VDD_PIC: no longer J3.2
Routing:
- net VDD_PIC: track 135.2 -> 132.0 mm
Changed lines of the file:
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@@
 <layer number="42" name="bRestrict" color="1" fill="10" visible="no" active="yes"/>
 <layer number="43" name="vRestrict" color="2" fill="10" visible="no" active="yes"/>
-<layer number="44" name="Drills" color="7" fill="1" visible="no" active="yes"/>
-<layer number="45" name="Holes" color="7" fill="1" visible="yes" active="yes"/>
-<layer number="46" name="Milling" color="3" fill="1" visible="no" active="yes"/>
+<layer number="44" name="Drills" color="14" fill="1" visible="yes" active="yes"/>
+<layer number="45" name="Holes" color="12" fill="1" visible="yes" active="yes"/>
+<layer number="46" name="Milling" color="3" fill="1" visible="yes" active="yes"/>
 <layer number="47" name="Measures" color="7" fill="1" visible="no" active="yes"/>
 <layer number="48" name="Document" color="7" fill="1" visible="yes" active="yes"/>
@@
 <rectangle x1="52.07" y1="20.955" x2="54.61" y2="26.035" layer="41"/>
 <rectangle x1="59.69" y1="12.065" x2="62.23" y2="17.145" layer="41"/>
-<hole x="17.78" y="46.355" drill="6.3754"/>
+<hole x="17.78" y="45.085" drill="6.3754"/>
 <rectangle x1="71.755" y1="24.13" x2="98.425" y2="25.4" layer="43"/>
 <rectangle x1="88.9" y1="0" x2="99.06" y2="21.59" layer="43"/>
@@
 <attribute name="NAME" x="27.686" y="27.305" size="1.27" layer="25" ratio="10" rot="R270"/>
 </element>
-<element name="F1" library="SparkFun" package="PTC-1206" value="1A PTC" x="29.21" y="29.21" rot="R180">
-<attribute name="IHOLD" value="500 mA" x="29.21" y="29.21" size="1.778" layer="27" rot="R180" display="off"/>
-<attribute name="ITRIP" value="1A" x="29.21" y="29.21" size="1.778" layer="27" rot="R180" display="off"/>
-<attribute name="DIGIKEY" value="F3733CT-ND" x="29.21" y="29.21" size="1.778" layer="27" rot="R180" display="off"/>
+<element name="F1" library="SparkFun" package="PTC-1206" value="2.2A PTC" x="29.21" y="29.21" rot="R180">
+<attribute name="IHOLD" value="1.10 A" x="29.21" y="29.21" size="1.778" layer="27" rot="R180" display="off"/>
+<attribute name="ITRIP" value="2.2A" x="29.21" y="29.21" size="1.778" layer="27" rot="R180" display="off"/>
+<attribute name="DIGIKEY" value="F3366CT-ND" x="29.21" y="29.21" size="1.778" layer="27" rot="R180" display="off"/>
 </element>
 </elements>
@@
 <wire x1="14.735" y1="34.42" x2="13.335" y2="33.02" width="0.3048" layer="1"/>
 <wire x1="99.06" y1="50.165" x2="97.155" y2="50.165" width="0.3048" layer="1"/>
-<wire x1="97.155" y1="50.165" x2="97.155" y2="50.45" width="0" layer="19" extent="1-1"/>
 </signal>
 <signal name="OSC1">
@@
 <via x="38.735" y="77.47" extent="1-16" drill="0.6096"/>
 <via x="63.5" y="63.5" extent="1-16" drill="0.6096"/>
-<contactref element="J3" pad="2"/>
-<wire x1="48.26" y1="77.47" x2="48.26" y2="80.645" width="0.254" layer="16"/>
 </signal>
 <signal name="UART_RX">
@@
 <wire x1="21.59" y1="51.435" x2="12.7" y2="51.435" width="0.3048" layer="16"/>
 <contactref element="U$5" pad="1"/>
-<wire x1="12.7" y1="53.34" x2="12.7" y2="52.07" width="0.3048" layer="1"/>
-<wire x1="12.7" y1="52.07" x2="12.7" y2="51.435" width="0.3048" layer="1"/>
-<wire x1="12.7" y1="43.18" x2="7.62" y2="38.1" width="0.254" layer="1"/>
-<wire x1="12.7" y1="52.07" x2="12.7" y2="43.18" width="0.254" layer="1"/>
+<wire x1="12.7" y1="53.34" x2="12.7" y2="51.435" width="0.3048" layer="1"/>
 <wire x1="7.62" y1="38.1" x2="7.62" y2="37.51" width="0.254" layer="1"/>
 <wire x1="26.67" y1="36.83" x2="27.94" y2="36.83" width="0.254" layer="16"/>
@@
 <wire x1="30.6578" y1="36.3728" x2="30.48" y2="36.195" width="0.3048" layer="1"/>
 <wire x1="30.48" y1="36.195" x2="27.94" y2="36.195" width="0.3048" layer="1"/>
+<wire x1="12.7" y1="51.435" x2="12.7" y2="50.165" width="0.3048" layer="1"/>
+<wire x1="12.7" y1="50.165" x2="7.62" y2="45.085" width="0.3048" layer="1"/>
+<wire x1="7.62" y1="45.085" x2="7.62" y2="37.465" width="0.3048" layer="1"/>
 <wire x1="30.6578" y1="36.3728" x2="30.6578" y2="36.195" width="0" layer="19" extent="1-1"/>
+<wire x1="7.62" y1="37.51" x2="7.62" y2="37.465" width="0" layer="19" extent="1-1"/>
 </signal>
 <signal name="N$6">
@@
 <wire x1="30.48" y1="29.21" x2="30.61" y2="29.21" width="0.254" layer="1"/>
 </signal>
+<signal name="PICKIT-VDD">
+<contactref element="J3" pad="2"/>
+</signal>
 </signals>

Commit message: changed project requirements document
Parts:
- R1: value 500 -> 510
Routing:
- net VDD_MIWI: track 51.0 -> 50.4 mm
Changed lines of the file:
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@@
 <layer number="42" name="bRestrict" color="1" fill="10" visible="no" active="yes"/>
 <layer number="43" name="vRestrict" color="2" fill="10" visible="no" active="yes"/>
-<layer number="44" name="Drills" color="14" fill="1" visible="yes" active="yes"/>
-<layer number="45" name="Holes" color="12" fill="1" visible="yes" active="yes"/>
-<layer number="46" name="Milling" color="3" fill="1" visible="yes" active="yes"/>
+<layer number="44" name="Drills" color="14" fill="1" visible="no" active="yes"/>
+<layer number="45" name="Holes" color="12" fill="1" visible="no" active="yes"/>
+<layer number="46" name="Milling" color="3" fill="1" visible="no" active="yes"/>
 <layer number="47" name="Measures" color="7" fill="1" visible="no" active="yes"/>
 <layer number="48" name="Document" color="7" fill="1" visible="yes" active="yes"/>
@@
 </element>
 <element name="C1" library="4534_I2C2" package="C2.5-5" value="10uF" x="40.64" y="37.465" rot="R90"/>
-<element name="C2" library="4534_I2C2" package="C2.5-5" value="10uF" x="27.94" y="37.465" rot="R90"/>
+<element name="C2" library="4534_I2C2" package="C2.5-5" value="10uF" x="27.94" y="37.465" smashed="yes" rot="R90">
+<attribute name="NAME" x="26.67" y="40.005" size="1.27" layer="25" font="vector" ratio="15"/>
+<attribute name="VALUE" x="30.48" y="34.925" size="1.27" layer="27" font="vector" ratio="15" rot="R180"/>
+</element>
 <element name="REG2" library="4534_Node_Board" package="SOIC8-N_MC" value="MCP1725-XXXXX/SN" x="60.96" y="14.605">
 <attribute name="NEWARK" value="MCP1725-3002E/SN" x="157.48" y="-107.315" size="1.778" layer="27" display="off"/>
@@
 <attribute name="VALUE" x="9.525" y="77.343" size="1.27" layer="27"/>
 </element>
-<element name="R1" library="4534_I2C2" package="R1206" value="500" x="22.86" y="74.295" smashed="yes" rot="R90">
+<element name="R1" library="4534_I2C2" package="R1206" value="510" x="22.86" y="74.295" smashed="yes" rot="R90">
 <attribute name="NAME" x="21.59" y="73.66" size="1.27" layer="25" font="vector" ratio="15" rot="R90"/>
 <attribute name="VALUE" x="25.4" y="73.025" size="1.27" layer="27" font="vector" ratio="15" rot="R90"/>
@@
 <wire x1="30.48" y1="77.47" x2="29.21" y2="76.2" width="0.254" layer="1"/>
 <wire x1="38.735" y1="77.47" x2="30.48" y2="77.47" width="0.254" layer="1"/>
-<wire x1="58.42" y1="77.47" x2="48.26" y2="77.47" width="0.254" layer="16"/>
-<wire x1="48.26" y1="77.47" x2="38.735" y2="77.47" width="0.254" layer="16"/>
+<wire x1="58.42" y1="77.47" x2="38.735" y2="77.47" width="0.254" layer="16"/>
 <wire x1="63.5" y1="72.39" x2="58.42" y2="77.47" width="0.254" layer="16"/>
 <wire x1="63.5" y1="63.5" x2="63.5" y2="72.39" width="0.254" layer="16"/>
@@
 <contactref element="U$5" pad="1"/>
 <wire x1="12.7" y1="53.34" x2="12.7" y2="51.435" width="0.3048" layer="1"/>
-<wire x1="7.62" y1="38.1" x2="7.62" y2="37.51" width="0.254" layer="1"/>
 <wire x1="26.67" y1="36.83" x2="27.94" y2="36.83" width="0.254" layer="16"/>
 <wire x1="24.13" y1="39.37" x2="26.67" y2="36.83" width="0.254" layer="16"/>
@@
 <wire x1="12.7" y1="51.435" x2="12.7" y2="50.165" width="0.3048" layer="1"/>
 <wire x1="12.7" y1="50.165" x2="7.62" y2="45.085" width="0.3048" layer="1"/>
-<wire x1="7.62" y1="45.085" x2="7.62" y2="37.465" width="0.3048" layer="1"/>
+<wire x1="7.62" y1="45.085" x2="7.62" y2="38.1" width="0.3048" layer="1"/>
+<wire x1="7.62" y1="38.1" x2="7.62" y2="37.51" width="0.3048" layer="1"/>
+<wire x1="7.62" y1="37.51" x2="7.62" y2="37.465" width="0.3048" layer="1"/>
 <wire x1="30.6578" y1="36.3728" x2="30.6578" y2="36.195" width="0" layer="19" extent="1-1"/>
-<wire x1="7.62" y1="37.51" x2="7.62" y2="37.465" width="0" layer="19" extent="1-1"/>
 </signal>
 <signal name="N$6">
