File: board_design/Spring12_6_rev4/Spring12_6_rev4.sch (EAGLE design)
At the start: 48 parts, among them IC1 LM555D, J3 PICKIT, Q1 20MHz, SW0 SW-PB-MOM

Commit message: board design... hopefully done
Parts:
- added C15: 100pF, rcl:C-USC1206
- added F1: 1A PTC, SparkFun:PTCSMD
- added J1, J2: (no value), 4534:MA07-1
- added L1: 10nH, rcl:L-USL1812
- added POWER: MA02-1, 4534:MA02-1
- added SV3, SV4, SV5: (no value), 4534:MA03-1
- added U$3, U$4, U$5: VIA, 4534_I2C2:VIA
- R5, R6: value 4K7 -> 10K
- U$2: value NHD-C0216CIZ-FN-FBW-3V -> NHD-C0216CIZ-FSW-FBW-3V3
Connections:
- removed net 5V: J3.2
- new net BATT: BATT0.VCC, F1.2
- new net CURRENT: J2.3, J2.4, J2.5, SV3.1, SV4.1, SV5.1
- new net MIWI-VDD: C15.1, L1.1, RF0.VIN
- new net N$12: F1.1, POWER.1
- new net N$14: J1.2
- new net N$17: J2.6
- new net N$21: J2.2
- new net N$7: J1.6
- new net VCC_REG0: C5.1, REG0.*SHDN, REG0.VIN, REG0.VIN_2, SV3.2
- new net VCC_REG1: C1.1, REG1.*SHDN, REG1.VIN, REG1.VIN_2, SV4.2
- new net VCC_REG2: C3.1, REG2.*SHDN, REG2.VIN, REG2.VIN_2, SV5.2
- net VCC_BATT: now also J1.3, J1.4, J1.5, POWER.2, SV3.3, SV4.3, SV5.3; no longer BATT0.VCC, C1.1, C3.1, C5.1, REG0.*SHDN, REG0.VIN, REG0.VIN_2, REG1.*SHDN, REG1.VIN, REG1.VIN_2, REG2.*SHDN, REG2.VIN, REG2.VIN_2
- net VDD_ACC: now also U$2.VDD, U$3.P, U$4.P
- net VDD_MIWI: now also L1.2, U$5.P; no longer RF0.VIN
- net VDD_PIC: now also J3.2; no longer U$2.VDD
- net VSS: now also C15.2, J1.1, J1.7, J2.1, J2.7

Commit message: more PCB revs
Parts:
- F1: value 1A PTC -> 2.2A PTC; DIGIKEY F3733CT-ND -> F3366CT-ND; IHOLD 500 mA -> 1.10 A; ITRIP 1A -> 2.2A
Connections:
- new net PICKIT-VDD: J3.2
- net VDD_PIC: no longer J3.2
Changed lines of the file:
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@@
 </part>
 <part name="POWER" library="4534" deviceset="MA02-1" device=""/>
-<part name="F1" library="SparkFun" deviceset="PTC" device="SMD" value="1A PTC">
-<attribute name="DIGIKEY" value="F3733CT-ND"/>
-<attribute name="IHOLD" value="500 mA"/>
-<attribute name="ITRIP" value="1A"/>
+<part name="F1" library="SparkFun" deviceset="PTC" device="SMD" value="2.2A PTC">
+<attribute name="DIGIKEY" value="F3366CT-ND"/>
+<attribute name="IHOLD" value="1.10 A"/>
+<attribute name="ITRIP" value="2.2A"/>
 </part>
 </parts>
@@
 <junction x="-53.34" y="187.96"/>
 </segment>
-<segment>
-<wire x1="-58.42" y1="50.8" x2="-86.36" y2="50.8" width="0.1524" layer="91"/>
-<label x="-81.28" y="50.8" size="1.778" layer="95"/>
-<pinref part="J3" gate="1" pin="2"/>
-</segment>
 </net>
 <net name="UART_RX" class="0">
@@
 </segment>
 </net>
+<net name="PICKIT-VDD" class="0">
+<segment>
+<pinref part="J3" gate="1" pin="2"/>
+<wire x1="-58.42" y1="50.8" x2="-86.36" y2="50.8" width="0.1524" layer="91"/>
+<label x="-81.28" y="50.8" size="1.778" layer="95"/>
+</segment>
+</net>

Commit message: changed project requirements document
Parts:
- R1: value 500 -> 510
Other:
- note added: "NC"
Changed lines of the file:
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@@
 <part name="U$20" library="4534_I2C2" deviceset="VIA" device=""/>
 <part name="IC1" library="4534" deviceset="*555" device="D" technology="LM"/>
-<part name="R1" library="4534_I2C2" deviceset="R1206" device="" value="500"/>
+<part name="R1" library="4534_I2C2" deviceset="R1206" device="" value="510"/>
 <part name="R2" library="4534_I2C2" deviceset="R1206" device="" value="1k"/>
 <part name="C14" library="4534_I2C2" deviceset="C2.5-5" device="" value="10uF"/>
@@
 <text x="5.08" y="226.06" size="1.778" layer="91">duty % = (R1 + R2) / (R1 + 2*R2)</text>
 <text x="-241.554" y="152.908" size="1.778" layer="91" rot="R180">~OE</text>
+<text x="-40.64" y="228.6" size="1.778" layer="91">NC</text>
 </plain>
 <instances>
